File: hardware/mcu.kicad_sch (KiCad schematic)
At the start: 1 part, among them IC1 SC1509

Commit message: XTR117 Output
Parts:
- removed IC1: SC1509, Samacsys:QFN40P700X700X90-61N-D, symbol Samacsys:SC1509
- added D1: D_Schottky, symbol Device:D_Schottky
- added J3: 24V_Terminal, symbol Connector:Screw_Terminal_01x02
- added U3: Pico, MCU_RaspberryPi_and_Boards:RPi_Pico_SMD_TH, symbol RP_Pico:Pico
Connections:
- new net +12V: D1.2 (A), J3.1 (Pin_1)
- new net +3V3_MCU: U3.36 (3V3)
- new net +5V_MCU: U3.40 (VBUS)
- new net GND_MCU: U3.3 (GND)
- new net GND_PSU: J3.2 (Pin_2)
- new net SPI0_CLK: U3.24 (GPIO18)
- new net SPI0_CS: U3.22 (GPIO17)
- new net SPI0_MISO: U3.21 (GPIO16)
- new net SPI0_MOSI: U3.25 (GPIO19)
- new net VSYS: D1.1 (K), U3.39 (VSYS)

Commit message: Almost everything
Parts:
- removed D1: D_Schottky, symbol Device:D_Schottky
- removed J3: 24V_Terminal, symbol Connector:Screw_Terminal_01x02
- added U29: DAC8562SDGSR, EasyEDA:VSSOP-10_L3.0-W3.0-P0.50-LS4.9-BL, symbol EasyEDA:DAC8562SDGSR
Connections:
- net SDA: now reaches U3.26 (GPIO20)
- net SCL: now reaches U3.27 (GPIO21)
- net ADC0: now reaches U3.31 (GPIO26_ADC0)
- net ADC1: now reaches U3.32 (GPIO27_ADC1)
- net DIN_2: now reaches U3.4 (GPIO2)
- net DIN_2: now also U3.5 (GPIO3)
- net DOUT_1: now reaches U3.6 (GPIO4)
- net DOOUT_2: now reaches U3.7 (GPIO5)
- net +3V3_MCU renamed +3V3
- net +5V_MCU: no longer names the net of U3.40 (VBUS)
- net SPI0_CLK renamed RS485_MODE
- net SPI0_CS renamed UART_RX
- net SPI0_MISO renamed UART_TX
- net SPI0_MOSI: no longer names the net of U3.25 (GPIO19)
- no-connect marks 0 -> 5
